File: mining/AXE/EdgeAxe.kicad_pcb (KiCad board)
At the start: 6 copper layers, 57 x 124.4 mm, 139 parts, among them J1 54-00164, J1 Conn_01x09_Male, J2 Conn_01x02, J2 Conn_01x09_Male, J3 Conn_01x05, J4 Conn_01x04, J5 TC2030-IDC, J7 Conn_01x02, J8 USB_C_Receptacle_USB2.0, J9 Conn_01x04, Q1 CSD17311Q5, Q2 CSD17311Q5, Q4 2N7002K, SW1 GT-TC029B-H025-L1N, SW2 GT-TC029B-H025-L1N, U1 25MHz, U1 Coral_1, U10 DS4432U+, U11 RT9080-33GJ5, U12 ESP32-S3-WROOM-1, U14 BM1366_mode1, U2 TXB0104RGYR, U5 MCP1824T-1802E, U6 MCP1824T-0802E, U7 EMC2101, U8 INA260, U9 TPS40305, Y1 32.768kHz

Commit message: cleanup
Parts:
- moved H7 23.9 mm to (130.0, 27.2)
- moved H8 23.8 mm to (80.4, 27.2)
Changed lines of the file:
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@@
 	(footprint "MountingHole:MountingHole_3mm_Pad_Via"
 		(layer "F.Cu")
-		(at 130.23501 51.12099)
+		(at 130 27.2)
 		(descr "Mounting Hole 3mm")
 		(tags "mounting hole 3mm")
@@
 	(footprint "MountingHole:MountingHole_3mm_Pad_Via"
 		(layer "F.Cu")
-		(at 80.35 51)
+		(at 80.4 27.2)
 		(descr "Mounting Hole 3mm")
 		(tags "mounting hole 3mm")
@@
 	)
 	(gr_text "BitcoinEDGE"
-		(at 128.8 43.6 -90)
+		(at 128.8 49.4 -90)
 		(layer "B.Cu")
 		(effects
@@
 	)
 	(gr_text "BitcoinEDGE"
-		(at 128.8 43.6 -90)
+		(at 128.8 49.4 -90)
 		(layer "B.Mask")
 		(effects
@@
 		(polygon
 			(pts
-				(xy 134.076661 51.386028) (xy 134.121 143.243) (xy 130.211 147.566) (xy 56.6 147.8) (xy 53.8 145.2)
-				(xy 53.8 49.8) (xy 56.2 47.2) (xy 129.914 47.209)
+				(xy 134.076661 51.386028) (xy 134.121 143.243) (xy 130.211 147.566) (xy 78.4 147.6) (xy 76.6 144.4)
+				(xy 76.4 54.8) (xy 76.4 50) (xy 134.2 49.8)
 			)
 		)
